File: KiCad files/Plasma Voltage Divider Opto-Isolator.kicad_pcb (KiCad board)
At the start: 2 copper layers, 142 x 43.2 mm, 24 parts, among them J1 Plasma Positive Work, J2 Power / Output, J3 Plasma Negative Electrode, U1 LM358, U2 HCNR200, U3 LM358

Commit message: Add files via upload
Other:
- board text added: "30mH"
- board text removed: "30MH"
Changed lines of the file:
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@@
       (outputformat 1)
       (mirror false)
-      (drillshape 1)
+      (drillshape 0)
       (scaleselection 1)
       (outputdirectory "")
@@
     (effects (font (size 1 1) (thickness 0.15)))
   )
-  (gr_text "30MH" (at 123 112.5) (layer "F.SilkS")
+  (gr_text "30mH" (at 123 112.5) (layer "F.SilkS")
     (effects (font (size 1 1) (thickness 0.15)))
   )
-  (gr_text "30MH" (at 123.25 80.5) (layer "F.SilkS")
+  (gr_text "30mH" (at 123.25 80.5) (layer "F.SilkS")
     (effects (font (size 1 1) (thickness 0.15)))
   )
