File: KiCad files/Plasma Voltage Divider Opto-Isolator.kicad_sch (KiCad schematic)
At the start: 24 parts, among them J1 Plasma Positive Work, J2 Power / Output, J3 Plasma Negative Electrode, U1 LM358, U2 HCNR200, U3 LM358

Commit message: Add files via upload
Parts:
- L1, L2: value 9x12 - 30MH -> 9x12 - 30mH
Changed lines of the file:
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@@
     (in_bom yes) (on_board yes)
     (property "Reference" "L1" (id 0) (at 83.566 96.266 90))
-    (property "Value" "9x12 - 30MH" (id 1) (at 83.566 98.806 90))
+    (property "Value" "9x12 - 30mH" (id 1) (at 83.566 98.806 90))
     (property "Footprint" "Inductor_THT:L_Radial_D9.5mm_P5.00mm_Fastron_07HVP" (id 2) (at 83.312 102.108 0)
       (effects (font (size 1.27 1.27)) hide)
@@
     (in_bom yes) (on_board yes)
     (property "Reference" "L2" (id 0) (at 83.312 120.142 90))
-    (property "Value" "9x12 - 30MH" (id 1) (at 83.566 118.11 90))
+    (property "Value" "9x12 - 30mH" (id 1) (at 83.566 118.11 90))
     (property "Footprint" "Inductor_THT:L_Radial_D9.5mm_P5.00mm_Fastron_07HVP" (id 2) (at 83.312 114.808 0)
       (effects (font (size 1.27 1.27)) hide)
@@
     )
     (path "/06ee30f1-5d18-40d9-866a-8ff53a99afdb"
-      (reference "L1") (unit 1) (value "9x12 - 30MH") (footprint "Inductor_THT:L_Radial_D9.5mm_P5.00mm_Fastron_07HVP")
+      (reference "L1") (unit 1) (value "9x12 - 30mH") (footprint "Inductor_THT:L_Radial_D9.5mm_P5.00mm_Fastron_07HVP")
     )
     (path "/0b937146-a7ec-4e8d-88a4-4f9c9211f808"
-      (reference "L2") (unit 1) (value "9x12 - 30MH") (footprint "Inductor_THT:L_Radial_D9.5mm_P5.00mm_Fastron_07HVP")
+      (reference "L2") (unit 1) (value "9x12 - 30mH") (footprint "Inductor_THT:L_Radial_D9.5mm_P5.00mm_Fastron_07HVP")
     )
     (path "/96005b21-5413-4f05-b50c-80d0bb576133"
